File: H23R30/Design/H23R30.brd (EAGLE design)
At the start: 34.6 x 30 mm, 33 parts, among them P1 HEXABIT_17.32_NO_P4_P10_P11, U1 STM32F091CBU6, U2 BLUENRG-M2SA, X1 XTALL_CSTCE8M00G52

Commit message: Release REV 1
Other:
- board text added: "H23R31"
- board text removed: "H23R30"
Changed lines of the file:
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@@
 <drawing>
 <settings>
-<setting alwaysvectorfont="no"/>
+<setting alwaysvectorfont="yes"/>
 <setting verticaltext="up"/>
 </settings>
@@
 <layer number="23" name="tOrigins" color="15" fill="1" visible="no" active="yes"/>
 <layer number="24" name="bOrigins" color="15" fill="1" visible="no" active="yes"/>
-<layer number="25" name="tNames" color="7" fill="1" visible="no" active="yes"/>
+<layer number="25" name="tNames" color="7" fill="1" visible="yes" active="yes"/>
 <layer number="26" name="bNames" color="7" fill="1" visible="yes" active="yes"/>
 <layer number="27" name="tValues" color="7" fill="1" visible="no" active="yes"/>
@@
 <text x="34.62" y="46.78" size="1.9304" layer="21" font="vector" align="center">P5</text>
 <text x="34.62" y="46.78" size="1.9304" layer="22" font="vector" rot="MR0" align="center">P5</text>
-<text x="34.6964" y="25.550875" size="1.9304" layer="22" font="vector" rot="MR180" align="center">H23R30</text>
+<text x="34.6964" y="25.550875" size="1.9304" layer="22" font="vector" rot="MR180" align="center">H23R31</text>
 <rectangle x1="40.64126875" y1="33.582103125" x2="40.656" y2="33.596834375" layer="21"/>
 <rectangle x1="40.523415625" y1="33.596834375" x2="40.670734375" y2="33.611565625" layer="21"/>
@@
 <attribute name="MFN" value="STMicroelectronics" x="28.2448" y="30.9372" size="1.778" layer="27" rot="R120" display="off"/>
 <attribute name="MPN" value="BlueNRG_M2SA" x="28.2448" y="30.9372" size="1.778" layer="27" rot="R120" display="off"/>
-<attribute name="NAME" x="23.855728125" y="22.5372875" size="1.27" layer="25" rot="R120"/>
+<attribute name="NAME" x="26.141728125" y="26.0932875" size="1.27" layer="25" rot="R120"/>
 <attribute name="OCTOPART_URL" value="https://octopart.com/bluenrg-m2sa-stmicroelectronics-104772812?r=sp" x="28.2448" y="30.9372" size="1.778" layer="27" rot="R120" display="off"/>
 <attribute name="VALUE" x="37.16394375" y="30.220790625" size="1.27" layer="27" rot="R120"/>
@@
 <attribute name="MFN" value="KEMET" x="20.7772" y="37.0332" size="1.778" layer="27" rot="R30" display="off"/>
 <attribute name="MPN" value="C0603C104K8RACTU" x="20.7772" y="37.0332" size="1.778" layer="27" rot="R30" display="off"/>
-<attribute name="NAME" x="20.519371875" y="38.256228125" size="1.016" layer="25" rot="R30"/>
+<attribute name="NAME" x="20.392371875" y="38.129228125" size="1.016" layer="25" rot="R30"/>
 <attribute name="OCTOPART_URL" value="https://octopart.com/c0603c104k8ractu-kemet-145075?r=sp&amp;s=9bS9ASSwSEqMCE9KBEQZ0g" x="20.7772" y="37.0332" size="1.778" layer="27" rot="R30" display="off"/>
 <attribute name="TOLERANCE" value="10%" x="20.7772" y="37.0332" size="1.778" layer="27" rot="R30" display="off"/>

Commit message: Fix To REV0
Other:
- board text added: "H23R30"
- board text removed: "H23R31"
Changed lines of the file:
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@@
 <text x="34.62" y="46.78" size="1.9304" layer="21" font="vector" align="center">P5</text>
 <text x="34.62" y="46.78" size="1.9304" layer="22" font="vector" rot="MR0" align="center">P5</text>
-<text x="34.6964" y="25.550875" size="1.9304" layer="22" font="vector" rot="MR180" align="center">H23R31</text>
+<text x="34.6964" y="25.550875" size="1.9304" layer="22" font="vector" rot="MR180" align="center">H23R30</text>
 <rectangle x1="40.64126875" y1="33.582103125" x2="40.656" y2="33.596834375" layer="21"/>
 <rectangle x1="40.523415625" y1="33.596834375" x2="40.670734375" y2="33.611565625" layer="21"/>
