File: H23R30/Design/H23R30.sch (EAGLE design)
At the start: 21 parts, among them P1 HEXABIT_17.32_NO_P4_P10_P11, U1 STM32F091CBU6, X1 XTALL_CSTCE8M00G52

Commit message: Bluetooth BlueNRG module
Parts:
- added BB, BC, BD, BR, RXD, TXD: PAD4, HEXABITZ_CONNECTION_PARTS:PAD4
- added C10: 4.7uF, HEXABITZ_RCLS:C-0805-POL
- added C11, C12: 100nF, HEXABITZ_RCLS:C-0603
- added R4: 10.0K, HEXABITZ_RCLS:R-0603
- added R5: 4.7K, HEXABITZ_RCLS:R-0603
- added U2: BLUENRG-M2SA, HEXABITZ_ICs:BLUENRG-M2SA
Connections:
- new net B2: BB.P$1, R4.2, U2.BOOT/DIO7
- new net N$1: BD.P$1, U2.SWDIO/DIO10
- new net N$2: BC.P$1, U2.SWCLK/DIO9
- new net N$8: BR.P$1, C12.2, R5.1, U2.RESETN
- net GND: now also C10.-, C11.2, C12.1, R4.1, U2.GND, U2.GND@1
- net UART1_RX: now also P1.SD5
- net UART1_TX: now also P1.SU5
- net UART2_RX: now also P1.SD2
- net UART2_TX: now also P1.SU2
- net UART3_RX: now also TXD.P$1, U2.DIO5
- net UART3_TX: now also RXD.P$1, U2.DIO4
- net UART4_RX: now also P1.SD1
- net UART4_TX: now also P1.SU1
- net UART5_RX: now also P1.SD6
- net UART5_TX: now also P1.SU6
- net UART6_RX: now also P1.SD3
- net UART6_TX: now also P1.SU3
- net VDD: now also C10.+, C11.1, R5.2, U2.VIN
Other:
- note added: "BlueNRG-M2 Bluetooth Module"
- note removed: "Add Description Here"

Commit message: Release REV 1
Other:
- note removed: "0"
Changed lines of the file:
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@@
 <wire x1="168.91" y1="18.288" x2="168.91" y2="22.86" width="0.1524" layer="205"/>
 <text x="222.25" y="10.2108" size="1.9304" layer="101" font="vector">Letter</text>
-<text x="227.6602" y="14.7066" size="1.9304" layer="101" font="vector">0</text>
+<text x="227.6602" y="14.7066" size="1.9304" layer="101" font="vector">1</text>
 <text x="223.52" y="5.3848" size="1.9304" layer="101" font="vector">1</text>
 <text x="228.346" y="5.3848" size="1.9304" layer="101" font="vector">2</text>
@@
 <wire x1="168.91" y1="18.288" x2="168.91" y2="22.86" width="0.1524" layer="205"/>
 <text x="222.25" y="10.2108" size="1.9304" layer="101" font="vector">Letter</text>
-<text x="227.6602" y="14.7066" size="1.9304" layer="101" font="vector">0</text>
+<text x="227.6602" y="14.7066" size="1.9304" layer="101" font="vector">1</text>
 <text x="223.52" y="5.3848" size="1.9304" layer="101" font="vector">2</text>
 <text x="228.346" y="5.3848" size="1.9304" layer="101" font="vector">2</text>

Commit message: Fix To REV0
Other:
- note added: "0"
- note added: "Salah Souda"
Changed lines of the file:
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@@
 <setting verticaltext="up"/>
 </settings>
-<grid distance="0.05" unitdist="inch" unit="inch" style="lines" multiple="1" display="no" altdistance="0.01" altunitdist="inch" altunit="inch"/>
+<grid distance="25" unitdist="mil" unit="mil" style="lines" multiple="1" display="no" altdistance="0.01" altunitdist="inch" altunit="inch"/>
 <layers>
 <layer number="1" name="Top" color="4" fill="1" visible="no" active="no"/>
@@
 <wire x1="168.91" y1="18.288" x2="168.91" y2="22.86" width="0.1524" layer="205"/>
 <text x="222.25" y="10.2108" size="1.9304" layer="101" font="vector">Letter</text>
-<text x="227.6602" y="14.7066" size="1.9304" layer="101" font="vector">1</text>
+<text x="227.6602" y="14.7066" size="1.9304" layer="101" font="vector">0</text>
 <text x="223.52" y="5.3848" size="1.9304" layer="101" font="vector">1</text>
 <text x="228.346" y="5.3848" size="1.9304" layer="101" font="vector">2</text>
@@
 <wire x1="231.14" y1="18.288" x2="231.14" y2="22.86" width="0.1524" layer="205"/>
 <text x="242.6462" y="6.1722" size="1.9304" layer="100" font="vector">www.hexabitz.com</text>
+<text x="184.7342" y="5.0292" size="1.9304" layer="101" font="vector">Salah Souda</text>
 </plain>
 <instances>
@@
 <wire x1="168.91" y1="18.288" x2="168.91" y2="22.86" width="0.1524" layer="205"/>
 <text x="222.25" y="10.2108" size="1.9304" layer="101" font="vector">Letter</text>
-<text x="227.6602" y="14.7066" size="1.9304" layer="101" font="vector">1</text>
+<text x="227.6602" y="14.7066" size="1.9304" layer="101" font="vector">0</text>
 <text x="223.52" y="5.3848" size="1.9304" layer="101" font="vector">2</text>
 <text x="228.346" y="5.3848" size="1.9304" layer="101" font="vector">2</text>
@@
 <text x="242.6462" y="6.1722" size="1.9304" layer="100" font="vector">www.hexabitz.com</text>
 <text x="111.76" y="107.95" size="1.778" layer="95">VDD Coupling</text>
+<text x="183.4642" y="5.0292" size="1.9304" layer="101" font="vector">Salah Souda</text>
 </plain>
 <instances>
